Commit message: add bumper sensor to end-effector. Collision detection with the ground

File: my_doosan_pkg/description/urdf/a0912.blue.urdf (robot description, URDF)
Before this commit: robot a0912, 8 links, 7 joints
Links:
- link base_0: mass 3.722 -> 3.635; geometry collision mesh filename=file:///$(find my_doosan_pkg)/description/meshes/a0912_blue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 scale=0.001 0.001 0.001; visual mesh filename=package://my_doosan_pkg/description/meshes/a0912_blue/A0912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 scale=0.001 0.001 0.001
- link link1: mass 7.446 -> 7.863; geometry collision cylinder length=0.2 radius=0.08; visual mesh filename=package://my_doosan_pkg/description/meshes/a0912_blue/A0912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 scale=0.001 0.001 0.001
- link link2: mass 10.569 -> 10.985; geometry collision cylinder length=0.6 radius=0.08; visual mesh filename=package://my_doosan_pkg/description/meshes/a0912_blue/A0912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 scale=0.001 0.001 0.001
- link link3: mass 3.614 -> 2.881
- link link4: mass 3.785 -> 3.273; geometry collision cylinder length=0.4 radius=0.05; visual mesh filename=package://my_doosan_pkg/description/meshes/a0912_blue/A0912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 scale=0.001 0.001 0.001
- link link5: mass 2.598 -> 2.141; geometry collision cylinder length=0.15 radius=0.06; visual mesh filename=package://my_doosan_pkg/description/meshes/a0912_blue/A0912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 scale=0.001 0.001 0.001
- link link6: mass 1.128 -> 0.784; geometry collision mesh filename=file:///$(find my_doosan_pkg)/description/meshes/a0912_blue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 scale=0.001 0.001 0.001; visual mesh filename=package://my_doosan_pkg/description/meshes/a0912_blue/A0912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 scale=0.001 0.001 0.001
Joints:
- joint joint1: limit lower=-2.617 upper=2.617 effort=30 velocity=1.571 -> lower=-6.2832 upper=6.2832 effort=411 velocity=3.1416
- joint joint2: limit lower=-2.617 upper=2.617 effort=30 velocity=1.571 -> lower=-6.2832 upper=6.2832 effort=411 velocity=3.1416
- joint joint3: limit lower=-2.617 upper=2.617 effort=30 velocity=1.571 -> lower=-2.7925 upper=2.7925 effort=194 velocity=3.1416
- joint joint4: limit lower=-2.617 upper=2.617 effort=30 velocity=1.571 -> lower=-6.2832 upper=6.2832 effort=50 velocity=6.2832
- joint joint5: limit lower=-2.617 upper=2.617 effort=30 velocity=1.571 -> lower=-6.2832 upper=6.2832 effort=50 velocity=6.2832
- joint joint6: limit lower=-2.617 upper=2.617 effort=30 velocity=1.571 -> lower=-6.2832 upper=6.2832 effort=50 velocity=6.2832

File: my_doosan_pkg/description/xacro/macro.a0912.blue.xacro (robot description, xacro)
@@ -3,8 +3,10 @@
 	<!-- I did some modifications concerning the original file-->
 	<!-- The  damping and friction where added in each joint-->
-	<!-- The created addded, and called the gazebo_config_control.xacro -->
+	<!-- The created added, and called the gazebo_config_control.xacro -->
+	<!-- The created added, and called the bumper_config.xacro -->
 	<xacro:include filename="$(find my_doosan_pkg)/description/xacro/macro.gazebo_config_control.xacro" />
 	<xacro:include filename="$(find my_doosan_pkg)/description/xacro/macro.transmission.xacro" />
 	<xacro:include filename="$(find my_doosan_pkg)/description/xacro/macro.internal_config.xacro" />
+	<xacro:include filename="$(find my_doosan_pkg)/description/xacro/macro.bumper_config.xacro" />
 	<xacro:macro name="a0912" params="namespace">
 		<!-- Base -->
@@ -247,8 +249,10 @@
       		</collision>
 		</link>
-		<!-- the following lines instantiates all the info described in the file macro.gazebo_config_control.xacro, transmissions and internal_config by david-->
+		<!-- the following lines instantiates all the info described in the files:
+		 macro.gazebo_config_control.xacro, transmissions,  internal_config, macro.bumper_config  by david-->
 		<xacro:config_ctr_gazebo />
 		<xacro:dsr_transmission />
 		<xacro:dsr_config_coeff />
+		<xacro:bumper_ctr_sensor />
 	</xacro:macro>
 </robot>

File: my_doosan_pkg/description/xacro/macro.gazebo_config_control.xacro (robot description, xacro)
@@ -3,5 +3,5 @@
 	<xacro:macro name="config_ctr_gazebo">
 		<!-- I need this for ROS2 control -->
-		<!-- I create this file, it was not avaliable in the orginal doosan repo -->
+		<!-- I create this file, it was NOT available in the original Doosan repo -->
 		<ros2_control name="GazeboSystem" type="system">
 			<hardware>

File: my_doosan_pkg/description/xacro/macro.internal_config.xacro (robot description, xacro)
@@ -3,5 +3,5 @@
 	<xacro:macro name="dsr_config_coeff">
     <!-- I need this for a better simulation in Gazebo-->
-    <!-- I modificated this file a bit, it was  avaliable in the orginal doosan repo as macro.gazebo.xacro -->
+    <!-- I modified this file a bit, it was available in the original Doosan repo as macro.gazebo.xacro -->
     <!-- This include the Contact Coefficients and other parameters, still no sure if this is correct -->
     <!-- More info here http://gazebosim.org/tutorials?tut=ros_urdf -->
