Commit message: migrate and files need to work with new ROS2

File: my_doosan_pkg/description/xacro/macro.a0912.blue.xacro (robot description, xacro)
@@ -22,10 +22,10 @@
 				<origin rpy="0 0 0" xyz="0 0 0" />
 				<geometry>
-					<mesh filename="file:///$(find my_doosan_pkg)/description/meshes/a0912_blue/A0912_0_0.dae" scale="0.001 0.001 0.001" />
+					<mesh filename="file://$(find my_doosan_pkg)/description/meshes/a0912_blue/A0912_0_0.dae" scale="0.001 0.001 0.001" />
 				</geometry>
 			</visual>
 			<collision>
         		<geometry>
-					<mesh filename="file:///$(find my_doosan_pkg)/description/meshes/a0912_blue/A0912_0_0.dae" scale="0.001 0.001 0.001" />
+					<mesh filename="file://$(find my_doosan_pkg)/description/meshes/a0912_blue/A0912_0_0.dae" scale="0.001 0.001 0.001" />
         		</geometry>
       		</collision>
@@ -57,17 +57,17 @@
 				<origin rpy="0 0 0" xyz="0 0 0" />
 				<geometry>
-					<mesh filename="file:///$(find my_doosan_pkg)/description/meshes/a0912_blue/A0912_1_0.dae" scale="0.001 0.001 0.001" />
-				</geometry>
-			</visual>
-            <visual>
-				<origin rpy="0 0 0" xyz="0 0 0" />
-				<geometry>
-					<mesh filename="file:///$(find my_doosan_pkg)/description/meshes/a0912_blue/A0912_1_1.dae" scale="0.001 0.001 0.001" />
-				</geometry>
-			</visual>
-            <visual>
-				<origin rpy="0 0 0" xyz="0 0 0" />
-				<geometry>
-					<mesh filename="file:///$(find my_doosan_pkg)/description/meshes/a0912_blue/A0912_1_2.dae" scale="0.001 0.001 0.001" />
+					<mesh filename="file://$(find my_doosan_pkg)/description/meshes/a0912_blue/A0912_1_0.dae" scale="0.001 0.001 0.001" />
+				</geometry>
+			</visual>
+            <visual>
+				<origin rpy="0 0 0" xyz="0 0 0" />
+				<geometry>
+					<mesh filename="file://$(find my_doosan_pkg)/description/meshes/a0912_blue/A0912_1_1.dae" scale="0.001 0.001 0.001" />
+				</geometry>
+			</visual>
+            <visual>
+				<origin rpy="0 0 0" xyz="0 0 0" />
+				<geometry>
+					<mesh filename="file://$(find my_doosan_pkg)/description/meshes/a0912_blue/A0912_1_2.dae" scale="0.001 0.001 0.001" />
 				</geometry>
 			</visual>
@@ -99,17 +99,17 @@
 				<origin rpy="0 0 0" xyz="0 0 0" />
 				<geometry>
-					<mesh filename="file:///$(find my_doosan_pkg)/description/meshes/a0912_blue/A0912_2_0.dae" scale="0.001 0.001 0.001" />
-				</geometry>
-			</visual>
-			<visual>
-				<origin rpy="0 0 0" xyz="0 0 0" />
-				<geometry>
-					<mesh filename="file:///$(find my_doosan_pkg)/description/meshes/a0912_blue/A0912_2_1.dae" scale="0.001 0.001 0.001" />
-				</geometry>
-			</visual>
-			<visual>
-				<origin rpy="0 0 0" xyz="0 0 0" />
-				<geometry>
-					<mesh filename="file:///$(find my_doosan_pkg)/description/meshes/a0912_blue/A0912_2_2.dae" scale="0.001 0.001 0.001" />
+					<mesh filename="file://$(find my_doosan_pkg)/description/meshes/a0912_blue/A0912_2_0.dae" scale="0.001 0.001 0.001" />
+				</geometry>
+			</visual>
+			<visual>
+				<origin rpy="0 0 0" xyz="0 0 0" />
+				<geometry>
+					<mesh filename="file://$(find my_doosan_pkg)/description/meshes/a0912_blue/A0912_2_1.dae" scale="0.001 0.001 0.001" />
+				</geometry>
+			</visual>
+			<visual>
+				<origin rpy="0 0 0" xyz="0 0 0" />
+				<geometry>
+					<mesh filename="file://$(find my_doosan_pkg)/description/meshes/a0912_blue/A0912_2_2.dae" scale="0.001 0.001 0.001" />
 				</geometry>
 			</visual>
@@ -136,11 +136,11 @@
 				<origin rpy="0 0 0" xyz="0 0 0" />
 				<geometry>
-					<mesh filename="file:///$(find my_doosan_pkg)/description/meshes/a0912_blue/A0912_3_0.dae" scale="0.001 0.001 0.001" />
-				</geometry>
-			</visual>
-            <visual>
-				<origin rpy="0 0 0" xyz="0 0 0" />
-				<geometry>
-					<mesh filename="file:///$(find my_doosan_pkg)/description/meshes/a0912_blue/A0912_3_1.dae" scale="0.001 0.001 0.001" />
+					<mesh filename="file://$(find my_doosan_pkg)/description/meshes/a0912_blue/A0912_3_0.dae" scale="0.001 0.001 0.001" />
+				</geometry>
+			</visual>
+            <visual>
+				<origin rpy="0 0 0" xyz="0 0 0" />
+				<geometry>
+					<mesh filename="file://$(find my_doosan_pkg)/description/meshes/a0912_blue/A0912_3_1.dae" scale="0.001 0.001 0.001" />
 				</geometry>
 			</visual>
@@ -172,11 +172,11 @@
 				<origin rpy="0 0 0" xyz="0 0 0" />
 				<geometry>
-					<mesh filename="file:///$(find my_doosan_pkg)/description/meshes/a0912_blue/A0912_4_0.dae" scale="0.001 0.001 0.001" />
-				</geometry>
-			</visual>
-            <visual>
-				<origin rpy="0 0 0" xyz="0 0 0" />
-				<geometry>
-					<mesh filename="file:///$(find my_doosan_pkg)/description/meshes/a0912_blue/A0912_4_1.dae" scale="0.001 0.001 0.001" />
+					<mesh filename="file://$(find my_doosan_pkg)/description/meshes/a0912_blue/A0912_4_0.dae" scale="0.001 0.001 0.001" />
+				</geometry>
+			</visual>
+            <visual>
+				<origin rpy="0 0 0" xyz="0 0 0" />
+				<geometry>
+					<mesh filename="file://$(find my_doosan_pkg)/description/meshes/a0912_blue/A0912_4_1.dae" scale="0.001 0.001 0.001" />
 				</geometry>
 			</visual>
@@ -209,11 +209,11 @@
 				<origin rpy="0 0 0" xyz="0 0 0" />
 				<geometry>
-					<mesh filename="file:///$(find my_doosan_pkg)/description/meshes/a0912_blue/A0912_5_0.dae" scale="0.001 0.001 0.001" />
-				</geometry>
-			</visual>
-            <visual>
-				<origin rpy="0 0 0" xyz="0 0 0" />
-				<geometry>
-					<mesh filename="file:///$(find my_doosan_pkg)/description/meshes/a0912_blue/A0912_5_1.dae" scale="0.001 0.001 0.001" />
+					<mesh filename="file://$(find my_doosan_pkg)/description/meshes/a0912_blue/A0912_5_0.dae" scale="0.001 0.001 0.001" />
+				</geometry>
+			</visual>
+            <visual>
+				<origin rpy="0 0 0" xyz="0 0 0" />
+				<geometry>
+					<mesh filename="file://$(find my_doosan_pkg)/description/meshes/a0912_blue/A0912_5_1.dae" scale="0.001 0.001 0.001" />
 				</geometry>
 			</visual>
@@ -240,10 +240,10 @@
 				<origin rpy="0 0 0" xyz="0 0 0" />
 				<geometry>
-					<mesh filename="file:///$(find my_doosan_pkg)/description/meshes/a0912_blue/A0912_6_0.dae" scale="0.001 0.001 0.001" />
+					<mesh filename="file://$(find my_doosan_pkg)/description/meshes/a0912_blue/A0912_6_0.dae" scale="0.001 0.001 0.001" />
 				</geometry>
 			</visual>
 			<collision>
         		<geometry>
-          			<mesh filename="file:///$(find my_doosan_pkg)/description/meshes/a0912_blue/A0912_6_0.dae" scale="0.001 0.001 0.001" />
+          			<mesh filename="file://$(find my_doosan_pkg)/description/meshes/a0912_blue/A0912_6_0.dae" scale="0.001 0.001 0.001" />
         		</geometry>
       		</collision>
@@ -254,5 +254,6 @@
 		<xacro:dsr_transmission />
 		<xacro:dsr_config_coeff />
-		<xacro:bumper_ctr_sensor />
+		<!-- Phase 1: bumper (Classic gz contact plugin) disabled; migrated to gz contact sensor in Phase 3 -->
+		<!-- <xacro:bumper_ctr_sensor /> -->
 	</xacro:macro>
 </robot>

File: my_doosan_pkg/description/xacro/macro.gazebo_config_control.xacro (robot description, xacro)
@@ -4,7 +4,7 @@
 		<!-- I need this for ROS2 control -->
 		<!-- I create this file, it was NOT available in the original Doosan repo -->
-		<ros2_control name="GazeboSystem" type="system">
+		<ros2_control name="GazeboSimSystem" type="system">
 			<hardware>
-				<plugin>gazebo_ros2_control/GazeboSystem</plugin>
+				<plugin>gz_ros2_control/GazeboSimSystem</plugin>
 	    	</hardware>
 	    	<joint name="joint1">
@@ -64,7 +64,5 @@
 	  	</ros2_control>
 		<gazebo>
-			<plugin name="gazebo_ros2_control" filename="libgazebo_ros2_control.so">
-        		<!--<robot_sim_type>gazebo_ros2_control/DefaultRobotHWSim</robot_sim_type> -->
-				<robot_sim_type>gazebo_ros2_control/GazeboSystem</robot_sim_type>
+			<plugin filename="gz_ros2_control-system" name="gz_ros2_control::GazeboSimROS2ControlPlugin">
 				<parameters>$(find my_doosan_pkg)/config/simple_controller.yaml</parameters>
 		    </plugin>

File: my_doosan_pkg/description/xacro/macro.m1013.white.xacro (robot description, xacro)
@@ -19,10 +19,10 @@
 				<origin rpy="0 0 0" xyz="0 0 0" />
 				<geometry>
-					<mesh filename="file:///$(find my_doosan_pkg)/description/meshes/m1013_white/MF1013_0_0.dae" scale="0.001 0.001 0.001" />
+					<mesh filename="file://$(find my_doosan_pkg)/description/meshes/m1013_white/MF1013_0_0.dae" scale="0.001 0.001 0.001" />
 				</geometry>
 			</visual>
 			<collision>
         		<geometry>
-          			<mesh filename="file:///$(find my_doosan_pkg)/description/meshes/m1013_white/MF1013_0_0.dae" scale="0.001 0.001 0.001" />
+          			<mesh filename="file://$(find my_doosan_pkg)/description/meshes/m1013_white/MF1013_0_0.dae" scale="0.001 0.001 0.001" />
         		</geometry>
       		</collision>
@@ -54,5 +54,5 @@
 				<origin rpy="0 0 0" xyz="0 0 0" />
 				<geometry>
-					<mesh filename="file:///$(find my_doosan_pkg)/description/meshes/m1013_white/MF1013_1_0.dae" scale="0.001 0.001 0.001" />
+					<mesh filename="file://$(find my_doosan_pkg)/description/meshes/m1013_white/MF1013_1_0.dae" scale="0.001 0.001 0.001" />
 				</geometry>
 			</visual>
@@ -85,17 +85,17 @@
 				<origin rpy="0 0 0" xyz="0 0 0" />
 				<geometry>
-					<mesh filename="file:///$(find my_doosan_pkg)/description/meshes/m1013_white/MF1013_2_0.dae" scale="0.001 0.001 0.001" />
-				</geometry>
-			</visual>
-			<visual>
-				<origin rpy="0 0 0" xyz="0 0 0" />
-				<geometry>
-					<mesh filename="file:///$(find my_doosan_pkg)/description/meshes/m1013_white/MF1013_2_1.dae" scale="0.001 0.001 0.001" />
-				</geometry>
-			</visual>
-			<visual>
-				<origin rpy="0 0 0" xyz="0 0 0" />
-				<geometry>
-					<mesh filename="file:///$(find my_doosan_pkg)/description/meshes/m1013_white/MF1013_2_2.dae" scale="0.001 0.001 0.001" />
+					<mesh filename="file://$(find my_doosan_pkg)/description/meshes/m1013_white/MF1013_2_0.dae" scale="0.001 0.001 0.001" />
+				</geometry>
+			</visual>
+			<visual>
+				<origin rpy="0 0 0" xyz="0 0 0" />
+				<geometry>
+					<mesh filename="file://$(find my_doosan_pkg)/description/meshes/m1013_white/MF1013_2_1.dae" scale="0.001 0.001 0.001" />
+				</geometry>
+			</visual>
+			<visual>
+				<origin rpy="0 0 0" xyz="0 0 0" />
+				<geometry>
+					<mesh filename="file://$(find my_doosan_pkg)/description/meshes/m1013_white/MF1013_2_2.dae" scale="0.001 0.001 0.001" />
 				</geometry>
 			</visual>
@@ -122,11 +122,11 @@
 				<origin rpy="0 0 0" xyz="0 0 0" />
 				<geometry>
-					<mesh filename="file:///$(find my_doosan_pkg)/description/meshes/m1013_white/MF1013_3_0.dae" scale="0.001 0.001 0.001" />
-				</geometry>
-			</visual>
-			<collision>
-				<origin rpy="0 0 0" xyz="0 0 0" />
-				<geometry>
-					<mesh filename="file:///$(find my_doosan_pkg)/description/meshes/m1013_white/MF1013_3_0.dae" scale="0.001 0.001 0.001" />
+					<mesh filename="file://$(find my_doosan_pkg)/description/meshes/m1013_white/MF1013_3_0.dae" scale="0.001 0.001 0.001" />
+				</geometry>
+			</visual>
+			<collision>
+				<origin rpy="0 0 0" xyz="0 0 0" />
+				<geometry>
+					<mesh filename="file://$(find my_doosan_pkg)/description/meshes/m1013_white/MF1013_3_0.dae" scale="0.001 0.001 0.001" />
 				</geometry>
 			</collision>
@@ -158,11 +158,11 @@
 				<origin rpy="0 0 0" xyz="0 0 0" />
 				<geometry>
-					<mesh filename="file:///$(find my_doosan_pkg)/description/meshes/m1013_white/MF1013_4_0.dae" scale="0.001 0.001 0.001" />
-				</geometry>
-			</visual>
-			<visual>
-				<origin rpy="0 0 0" xyz="0 0 0" />
-				<geometry>
-					<mesh filename="file:///$(find my_doosan_pkg)/description/meshes/m1013_white/MF1013_4_1.dae" scale="0.001 0.001 0.001" />
+					<mesh filename="file://$(find my_doosan_pkg)/description/meshes/m1013_white/MF1013_4_0.dae" scale="0.001 0.001 0.001" />
+				</geometry>
+			</visual>
+			<visual>
+				<origin rpy="0 0 0" xyz="0 0 0" />
+				<geometry>
+					<mesh filename="file://$(find my_doosan_pkg)/description/meshes/m1013_white/MF1013_4_1.dae" scale="0.001 0.001 0.001" />
 				</geometry>
 			</visual>
@@ -195,5 +195,5 @@
 				<origin rpy="0 0 0" xyz="0 0 0" />
 				<geometry>
-					<mesh filename="file:///$(find my_doosan_pkg)/description/meshes/m1013_white/MF1013_5_0.dae" scale="0.001 0.001 0.001" />
+					<mesh filename="file://$(find my_doosan_pkg)/description/meshes/m1013_white/MF1013_5_0.dae" scale="0.001 0.001 0.001" />
 				</geometry>
 			</visual>
@@ -220,10 +220,10 @@
 				<origin rpy="0 0 0" xyz="0 0 0" />
 				<geometry>
-					<mesh filename="file:///$(find my_doosan_pkg)/description/meshes/m1013_white/MF1013_6_0.dae" scale="0.001 0.001 0.001" />
+					<mesh filename="file://$(find my_doosan_pkg)/description/meshes/m1013_white/MF1013_6_0.dae" scale="0.001 0.001 0.001" />
 				</geometry>
 			</visual>
 			<collision>
         		<geometry>
-          			<mesh filename="file:///$(find my_doosan_pkg)/description/meshes/m1013_white/MF1013_6_0.dae" scale="0.001 0.001 0.001" />
+          			<mesh filename="file://$(find my_doosan_pkg)/description/meshes/m1013_white/MF1013_6_0.dae" scale="0.001 0.001 0.001" />
         		</geometry>
       		</collision>
